File: electronics/onboard-systems/onboard-systems.kicad_sch (KiCad schematic)
At the start: 6 parts, among them SW1 GOOBAY_10013, U1 XIAO_ESP32_S3, U2 Adafruit_BMP580, U3 Adafruit_LSM6DSO32

Commit message: update models
Parts:
- removed SW1: GOOBAY_10013, GOOBAY:GOOBAY_10013, symbol GOOBAY:GOOBAY_10013
- removed TP-BAT-+1, TP2: TestPoint, TestPoint:TestPoint_Loop_D2.50mm_Drill1.85mm, symbol Connector:TestPoint
Connections:
- net GND: now also U3.14 (GND2)
